File: pico_w-valve-ctrl/pico_w-valve-ctrl.kicad_sch (KiCad schematic)
At the start: 8 parts

Commit message: addinf pico
Parts:
- added U?: Pico-MCU_RaspberryPi_and_Boards, RPi_Pico:RPi_Pico_SMD_TH, symbol pico-mcu_raspberrypi_and_boards:Pico-MCU_RaspberryPi_and_Boards
Changed lines of the file:
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@@
     (pin "2")
+  )
+  (symbol (lib_id "pico-mcu_raspberrypi_and_boards:Pico-MCU_RaspberryPi_and_Boards") (at 43.18 53.34 0) (unit 1)
+    (in_bom yes) (on_board yes) (fields_autoplaced)
+    (property "Reference" "U?" (id 0) (at 43.18 21.59 0))
+    (property "Value" "Pico-MCU_RaspberryPi_and_Boards" (id 1) (at 43.18 24.13 0))
+    (property "Footprint" "RPi_Pico:RPi_Pico_SMD_TH" (id 2) (at 43.18 53.34 90)
+      (effects (font (size 1.27 1.27)) hide)
+    )
+    (property "Datasheet" "" (id 3) (at 43.18 53.34 0)
+      (effects (font (size 1.27 1.27)) hide)
+    )
+    (pin "1")
+    (pin "10")
+    (pin "11")
+    (pin "12")
+    (pin "13")
+    (pin "14")
+    (pin "15")
+    (pin "16")
+    (pin "17")
+    (pin "18")
+    (pin "19")
+    (pin "2")
+    (pin "20")
+    (pin "21")
+    (pin "22")
+    (pin "23")
+    (pin "24")
+    (pin "25")
+    (pin "26")
+    (pin "27")
+    (pin "28")
+    (pin "29")
+    (pin "3")
+    (pin "30")
+    (pin "31")
+    (pin "32")
+    (pin "33")
+    (pin "34")
+    (pin "35")
+    (pin "36")
+    (pin "37")
+    (pin "38")
+    (pin "39")
+    (pin "4")
+    (pin "40")
+    (pin "41")
+    (pin "42")
+    (pin "43")
+    (pin "5")
+    (pin "6")
+    (pin "7")
+    (pin "8")
+    (pin "9")
   )
   (sheet_instances
@@
       (reference "R4") (unit 1) (value "330") (footprint "")
     )
+    (path "/fb8d182b-152b-496b-bfda-0e05563bbf0a"
+      (reference "U?") (unit 1) (value "Pico-MCU_RaspberryPi_and_Boards") (footprint "RPi_Pico:RPi_Pico_SMD_TH")
+    )
   )
